File: alpakka.kicad_sch (KiCad schematic)
At the start: 76 parts, among them P1 Debug, P2 Endpoint, P3 Conn_01x02, Q1 Q_PMOS_DGS, U1 Raspberry_Pico, U10 ST_LSM6, U12 ST_LSM6, U2 Alpsalpine_RKJXV, U3 Alpsalpine_EC10E, U4 Alpsalpine_RKJXM, U6 NXP_PCAL6416A, U8 NXP_PCAL6416A

Commit message: Changed JST connector, Added Mount and Export properties, Tweaked components origins
Parts:
- C1, C2, C3, C4, C5, C6, D1, D2, D3, D4, P2, R1, R2, R3, R4, R6, S1, S10, S11, S12, S14, S2, S3, S4, S5, S6, S7, S8, S9: Export (none) -> yes; Mount (none) -> SMD
- P1: footprint ILO_fp:Boomele_C50137 -> ILO_fp:JST_S4B-PH-SM4-K-TB; Export (none) -> yes; LCSC C50137 -> C265332; Mount (none) -> SMD
- S15, S16: LCSC (none) -> C125031; Mount (none) -> TH
- S17, S18, S19, S20: Export (none) -> yes; LCSC (none) -> C202424; Mount (none) -> SMD
- U1: LCSC (none) -> C7203002; Mount (none) -> SMD
- U10, U12: Export (none) -> yes; Group ARS -> IMU; Mount (none) -> SMD
- U2: LCSC (none) -> C918854; Mount (none) -> TH
- U3: LCSC (none) -> C110291; Mount (none) -> TH
- U4: LCSC (none) -> C97432; Mount (none) -> TH
- U6, U8: Export (none) -> yes; Group (none) -> IO; Mount (none) -> SMD
